Commit message: 20210503

File: demo/urdf/demo.urdf.xacro (robot description, xacro)
@@ -52,4 +52,21 @@
     <child link="mountingplate_link" />
   </joint>
+  <!-- Obstacle  -->
+<!--
+  <link name="obstacle_link">
+    <visual>
+      <origin xyz="0.005 0.02 0.1" />
+      <geometry>
+        <box size="0.01 0.4 0.2" />
+      </geometry>
+      <material name="blue"/>
+    </visual>
+  </link>
+  <joint name="obstacle_joint" type="fixed">
+    <origin xyz="0.0 0.15 0.021" />
+    <parent link="baseplate_link" />
+    <child link="obstacle_link" />
+  </joint>
+-->
   <!-- robot to mouting_plate. -->
   <joint name="mountingplate_to_robot_joint" type="fixed">
